File: 9x16/led_array.kicad_pcb (KiCad board)
At the start: 2 copper layers, 113.8 x 126.8 mm, 154 parts, among them M1 P***, M2 P***, M3 P***, M4 P***, P1 CONN_2, SW1 SWITCH_INV

Commit message: Modified design to a 9x18 LED array.
Parts:
- removed R4: R, R5
- added D145: LED, CUSTOM LED-5MM, F.Cu at (86.3, 147.5)
- added D146: LED, CUSTOM LED-5MM, F.Cu at (94.3, 147.5)
- added D147: LED, CUSTOM LED-5MM, F.Cu at (102.3, 147.5)
- added D148: LED, CUSTOM LED-5MM, F.Cu at (110.3, 147.5)
- added D149: LED, CUSTOM LED-5MM, F.Cu at (118.2, 147.5)
- added D150: LED, CUSTOM LED-5MM, F.Cu at (126.2, 147.5)
- added D151: LED, CUSTOM LED-5MM, F.Cu at (134.2, 147.5)
- added D152: LED, CUSTOM LED-5MM, F.Cu at (142.1, 147.5)
- added D153: LED, CUSTOM LED-5MM, F.Cu at (150.1, 147.5)
- added D154: LED, CUSTOM LED-5MM, F.Cu at (86.3, 155.5)
- added D155: LED, CUSTOM LED-5MM, F.Cu at (94.3, 155.5)
- added D156: LED, CUSTOM LED-5MM, F.Cu at (102.3, 155.5)
- added D157: LED, CUSTOM LED-5MM, F.Cu at (110.3, 155.5)
- added D158: LED, CUSTOM LED-5MM, F.Cu at (118.2, 155.5)
- added D159: LED, CUSTOM LED-5MM, F.Cu at (126.2, 155.5)
- added D160: LED, CUSTOM LED-5MM, F.Cu at (134.2, 155.5)
- added D161: LED, CUSTOM LED-5MM, F.Cu at (142.1, 155.5)
- added D162: LED, CUSTOM LED-5MM, F.Cu at (150.1, 155.5)
- moved M3 16.0 mm to (171.6, 155.4)
- moved M4 16.0 mm to (65.2, 155.4)
Connections:
- D1 pad 1: N-0000032 -> N-0000020
- D100 pad 2: N-0000031 -> N-0000089
- D101 pad 1: N-0000032 -> N-0000089
- D102 pad 2: N-0000010 -> N-0000036
- D103 pad 1: N-0000010 -> N-0000020
- D104 pad 2: N-0000031 -> N-0000082
- D105 pad 1: N-0000032 -> N-0000082
- D108 pad 2: N-0000031 -> N-0000036
- D109 pad 1: N-0000032 -> N-0000020
- D112 pad 2: N-0000029 -> N-000009
- D113 pad 1: N-0000032 -> N-000009
- D114 pad 2: N-0000075 (its old number) -> N-0000040
- D115 pad 1: N-0000075 (its old number) -> N-0000020
- D117 pad 1: N-0000032 -> N-0000029
- D12 pad 2: N-000005 (its old number) -> N-0000035
- D120 pad 2: N-0000029 -> N-0000040
- D121 pad 1: N-0000032 -> N-0000020
- D124 pad 2: N-0000029 -> N-000002
- D125 pad 1: N-0000032 -> N-000002
- D126 pad 2: N-0000089 -> N-0000040
- D127 pad 1: N-0000089 -> N-0000020
- D128 pad 2: N-0000029 -> N-0000044
- D129 pad 1: N-0000032 -> N-0000044
- D13 pad 1: N-0000032 -> N-0000020
- D132 pad 2: N-0000029 -> N-0000040
- D133 pad 1: N-0000032 -> N-0000020
- D136 pad 2: N-0000029 -> N-0000047
- D137 pad 1: N-0000032 -> N-0000047
- D138 pad 2: N-00000112 -> N-0000040
- D139 pad 1: N-00000112 -> N-0000020
- D140 pad 2: N-0000029 -> N-0000026
- D141 pad 1: N-0000032 -> N-0000026
- D144 pad 2: N-0000029 -> N-0000040
- D16 pad 2: N-000005 (its old number) -> N-00000106
- D17 pad 1: N-0000032 -> N-00000106
- D18 pad 2: N-0000054 (its old number) -> N-0000035
- D19 pad 1: N-0000054 (its old number) -> N-0000020
- D20 pad 2: N-000005 (its old number) -> N-00000128
- D21 pad 1: N-0000032 -> N-00000128
- D24 pad 2: N-000005 (its old number) -> N-0000035
- D25 pad 1: N-0000032 -> N-0000020
- D28 pad 2: N-000005 (its old number) -> N-0000076
- D29 pad 1: N-0000032 -> N-0000076
- D30 pad 2: N-0000048 (its old number) -> N-0000035
- D31 pad 1: N-0000048 (its old number) -> N-0000020
- D32 pad 2: N-000005 (its old number) -> N-0000073
- D33 pad 1: N-0000032 -> N-0000073
- D36 pad 2: N-000005 (its old number) -> N-0000035
- D37 pad 1: N-0000032 -> N-0000020
- D4 pad 2: N-000005 (its old number) -> N-00000112
- D40 pad 2: N-000004 (its old number) -> N-00000117
- D41 pad 1: N-0000032 -> N-00000117
- D42 pad 2: N-0000063 (its old number) -> N-0000035
- D43 pad 1: N-0000063 (its old number) -> N-0000020
- D44 pad 2: N-000004 (its old number) -> N-0000070
- D45 pad 1: N-0000032 -> N-0000070
- D48 pad 2: N-000004 (its old number) -> N-0000035
- D49 pad 1: N-0000032 -> N-0000020
- D5 pad 1: N-0000032 -> N-00000112
- D52 pad 2: N-000004 (its old number) -> N-00000100
- D53 pad 1: N-0000032 -> N-00000100
- D54 pad 2: N-0000036 -> N-0000035
- D55 pad 1: N-0000036 -> N-0000020
- D56 pad 2: N-000004 (its old number) -> N-0000097
- D57 pad 1: N-0000032 -> N-0000097
- D6 pad 2: N-0000099 (its old number) -> N-0000035
- D60 pad 2: N-000004 (its old number) -> N-0000036
- D61 pad 1: N-0000032 -> N-0000020
- D64 pad 2: N-000004 (its old number) -> N-0000091
- D65 pad 1: N-0000032 -> N-0000091
- D66 pad 2: N-0000061 (its old number) -> N-0000036
- D67 pad 1: N-0000061 (its old number) -> N-0000020
- D68 pad 2: N-000004 (its old number) -> N-0000094
- D69 pad 1: N-0000032 -> N-0000094
- D7 pad 1: N-0000099 (its old number) -> N-0000020
- D72 pad 2: N-000004 (its old number) -> N-0000036
- D73 pad 1: N-0000032 -> N-0000020
- D76 pad 2: N-0000031 -> N-0000052
- D77 pad 1: N-0000032 -> N-0000052
- D78 pad 2: N-0000021 -> N-0000036
- D79 pad 1: N-0000021 -> N-0000020
- D8 pad 2: N-000005 (its old number) -> N-00000125
- D80 pad 2: N-0000031 -> N-0000056
- D81 pad 1: N-0000032 -> N-0000056
- D84 pad 2: N-0000031 -> N-0000036
- D85 pad 1: N-0000032 -> N-0000020
- D88 pad 2: N-0000031 -> N-0000062
- D89 pad 1: N-0000032 -> N-0000062
- D9 pad 1: N-0000032 -> N-00000125
- D90 pad 2: N-0000016 (its old number) -> N-0000036
- D91 pad 1: N-0000016 (its old number) -> N-0000020
- D92 pad 2: N-0000031 -> N-0000059
- D93 pad 1: N-0000032 -> N-0000059
- D96 pad 2: N-0000031 -> N-0000036
- D97 pad 1: N-0000032 -> N-0000020
- R1 pad 1: N-000005 (its old number) -> N-0000035
- R2 pad 1: N-000004 (its old number) -> N-0000036
- R3 pad 1: N-0000031 -> N-0000040
- SW1 pad 2: N-0000032 -> N-0000020
Other:
- board size 113.8 x 126.8 mm -> 113.8 x 142.7 mm
- board text added: "IO Rodeo 9x18 LED Array v1.1"
- board text removed: "IO Rodeo 9x16 LED Array v1.1"
